File: crossover.kicad_sch (KiCad schematic)
At the start: 18 parts, among them J1 Connector, U7 LF356, U8 LF356

Commit message: Added JST
Parts:
- J1: footprint Connector_PinHeader_2.54mm:PinHeader_1x09_P2.54mm_Vertical -> Connector_JST:JST_PH_B9B-PH-K_1x09_P2.00mm_Vertical
Changed lines of the file:
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@@
 			)
 		)
-		(property "Footprint" "Connector_PinHeader_2.54mm:PinHeader_1x09_P2.54mm_Vertical"
+		(property "Footprint" "Connector_JST:JST_PH_B9B-PH-K_1x09_P2.00mm_Vertical"
 			(at 115.57 146.05 0)
 			(effects
